Commit message: Add wheel and fork offset to the forklift

File: data/forklift/forklift_robot.urdf (robot description, URDF)
Before this commit: robot forklift_robot, 6 links, 5 joints
Joints:
- joint base_to_fork: origin (none) -> xyz=2 0.2 0 rpy=0 0 0
- joint base_to_wheel_back_left: origin (none) -> xyz=0 .90 0 rpy=0 0 0
- joint base_to_wheel_back_right: origin (none) -> xyz=0 0 0 rpy=0 0 0
- joint base_to_wheel_front_left: origin (none) -> xyz=1.55 0.90 0 rpy=0 0 0
- joint base_to_wheel_front_right: origin (none) -> xyz=1.55 0 0 rpy=0 0 0
